File: ikea-fyrtur.kicad_pcb (KiCad board)
At the start: 4 copper layers, 44.5 x 22.5 mm, 46 parts, among them J1 EXT_CTRL, J2 MOTOR, J3 UART_TagConnect, J4 UART_2mm, J5 PWR, J6 I2C, J8 IO15, Q1 SS8050-G, Q2 SS8050-G, SW1 SW1_RST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

Commit message: - Change R9 from 1K to 120R (Setting GPIO0 line low via Down-Button may not lower voltage enough otherwise) - Added images, updated README - Change schematic revision to 0.71  (Resistor value change does not warrant change to the PCB)
Parts:
- R9: value 1K -> 120R
Changed lines of the file:
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@@
   (page A4)
   (layers
-    (0 F.Cu signal)
+    (0 F.Cu signal hide)
     (1 In1.Cu signal hide)
     (2 In2.Cu signal hide)
@@
       (effects (font (size 1 1) (thickness 0.15)))
     )
-    (fp_text user %R (at 0 0 90) (layer F.Fab)
-      (effects (font (size 1 1) (thickness 0.15)))
-    )
     (fp_line (start 3.9 2.25) (end 3.9 -3.25) (layer F.CrtYd) (width 0.05))
     (fp_line (start 2.3505 1.3335) (end -2.3495 1.3335) (layer F.SilkS) (width 0.12))
@@
     (fp_line (start 3.9 2.25) (end -3.9 2.25) (layer F.CrtYd) (width 0.05))
     (fp_line (start 3.9 -3.25) (end -3.9 -3.25) (layer F.CrtYd) (width 0.05))
+    (fp_text user %R (at 0 0 90) (layer F.Fab)
+      (effects (font (size 1 1) (thickness 0.15)))
+    )
     (pad "" np_thru_hole circle (at 0 -1.375 270) (size 0.75 0.75) (drill 0.7) (layers *.Cu *.Mask))
     (pad "" np_thru_hole circle (at 0 0.381 270) (size 0.75 0.75) (drill 0.7) (layers *.Cu *.Mask))
@@
     )
     (fp_text value S1 (at 0 3.5 90) (layer F.Fab)
-      (effects (font (size 1 1) (thickness 0.15)))
-    )
-    (fp_text user %R (at 0 0 90) (layer F.Fab)
       (effects (font (size 1 1) (thickness 0.15)))
     )
@@
     (fp_line (start 3.9 2.25) (end -3.9 2.25) (layer F.CrtYd) (width 0.05))
     (fp_line (start 3.9 -3.25) (end -3.9 -3.25) (layer F.CrtYd) (width 0.05))
+    (fp_text user %R (at 0 0 90) (layer F.Fab)
+      (effects (font (size 1 1) (thickness 0.15)))
+    )
     (pad "" np_thru_hole circle (at 0 -1.375 270) (size 0.75 0.75) (drill 0.7) (layers *.Cu *.Mask))
     (pad "" np_thru_hole circle (at 0 0.381 270) (size 0.75 0.75) (drill 0.7) (layers *.Cu *.Mask))
@@
       (effects (font (size 1 1) (thickness 0.15)) (justify mirror))
     )
-    (fp_text value 1K (at 0 -1.43) (layer B.Fab) hide
+    (fp_text value 120R (at 0 -1.43) (layer B.Fab) hide
       (effects (font (size 1 1) (thickness 0.15)) (justify mirror))
     )
@@
     (pad 1 thru_hole rect (at 0 0) (size 1.35 1.35) (drill 0.8) (layers *.Cu *.Mask)
       (net 6 GND))
-    (model ${KISYS3DMOD}/Connector_PinHeader_2.00mm.3dshapes/PinHeader_1x07_P2.00mm_Vertical.wrl
-      (at (xyz 0 0 0))
-      (scale (xyz 1 1 1))
-      (rotate (xyz 0 0 0))
-    )
   )
   (module RF_Module:ESP-12E locked (layer F.Cu)
